Commit message: end_point

File: src/robot_description/urdf/target.urdf (robot description, URDF)
Before this commit: robot with_craw, 15 links, 14 joints
Links:
- added link virtual_tip_link, mass 0.00001
Joints:
- added joint virtual_tip_joint: type revolute, parent craw_1, child virtual_tip_link, origin xyz= -0.1 -0.036 -0.00325 rpy=0 0 0, axis 0 0 1, limit lower=0 upper=0 effort=0 velocity=0

Commit message: cr5-v1

File: src/robot_description/urdf/target.urdf (robot description, URDF)
Before this commit: robot with_craw, 16 links, 15 joints
Joints:
- joint Revolute 3: limit (none) -> lower=-0.5236 upper=0.5236; type continuous -> revolute

Commit message: 123

File: src/robot_description/urdf/target.urdf (robot description, URDF)
Before this commit: robot with_craw, 16 links, 15 joints
Links:
- removed link 25joint_1
- removed link joint142_1
- removed link joint251_1
- removed link joint251_2
- removed link trans_1
- added link 14joint44v2_1, mass 6.462489586316137; collision mesh filename=package://robot_description/meshes/14joint44v2_1.stl scale=0.001 0.001 0.001; visual mesh filename=package://robot_description/meshes/14joint44v2_1.stl scale=0.001 0.001 0.001
- added link 25joint_v2_1, mass 15.540708623156803; collision mesh filename=package://robot_description/meshes/25joint_v2_1.stl scale=0.001 0.001 0.001; visual mesh filename=package://robot_description/meshes/25joint_v2_1.stl scale=0.001 0.001 0.001
- added link 25jointt_1, mass 15.540708623156789; collision mesh filename=package://robot_description/meshes/25jointt_1.stl scale=0.001 0.001 0.001; visual mesh filename=package://robot_description/meshes/25jointt_1.stl scale=0.001 0.001 0.001
- added link joint252_1, mass 15.540708623156794; collision mesh filename=package://robot_description/meshes/joint252_1.stl scale=0.001 0.001 0.001; visual mesh filename=package://robot_description/meshes/joint252_1.stl scale=0.001 0.001 0.001
- added link transv2_1, mass 9.761584230310485; collision mesh filename=package://robot_description/meshes/transv2_1.stl scale=0.001 0.001 0.001; visual mesh filename=package://robot_description/meshes/transv2_1.stl scale=0.001 0.001 0.001
- link base_link: mass 7.80323249079454 -> 7.803232490794544
- link board_1: mass 0.37239652270283546 -> 0.3723965227028356
- link cralwer_deap_1: mass 0.23667750006845437 -> 0.23667750006845484
- link craw_1: mass 2.0529823308563824 -> 2.052982330856382
- link crawler_deap12_1: mass 0.236677500068455 -> 0.2366775000684548
- link flange_1: mass 1.24878893227101 -> 1.2487889322710095
- link joint143_1: mass 6.4624895863161385 -> 6.462489586316132
- link joint14_1: mass 6.462489586316137 -> 6.462489586316139
Joints:
- removed joint Revolute 11
- removed joint Revolute 12
- removed joint Revolute 13
- removed joint Revolute 2
- removed joint Revolute 3
- removed joint Revolute 8
- removed joint Rigid 10
- removed joint Rigid 16
- removed joint Rigid 17
- removed joint Rigid 4
- removed joint Rigid 6
- removed joint Rigid 9
- removed joint Slider 19
- removed joint Slider 20
- added joint Revolute 21: type continuous, parent base_link, child joint252_1, origin xyz=0.001849 0.003782 0.07 rpy=0 0 0, axis 0.0 0.0 1.0
- added joint Revolute 22: type continuous, parent joint252_1, child 25joint_v2_1, origin xyz=0.0 -0.069999 0.076501 rpy=0 0 0, axis 0.0 -1.0 0.0
- added joint Revolute 34: type continuous, parent 25jointt_1, child transv2_1, origin xyz=0.0 0.071 0.066501 rpy=0 0 0, axis 0.0 -1.0 0.0
- added joint Revolute 40: type continuous, parent joint14_1, child 14joint44v2_1, origin xyz=0.0 -0.058 0.049 rpy=0 0 0, axis 0.0 -1.0 -0.0
- added joint Revolute 41: type continuous, parent 14joint44v2_1, child joint143_1, origin xyz=0.0 -0.049 0.058 rpy=0 0 0, axis 0.0 -0.0 1.0
- added joint Revolute 42: type continuous, parent joint143_1, child flange_1, origin xyz=0.0 -0.058 0.049 rpy=0 0 0, axis 0.0 -1.0 -0.0
- added joint Rigid 30: type fixed, parent 25joint_v2_1, child larm_1, origin xyz=0.0 -0.071 0.066501 rpy=0 0 0
- added joint Rigid 32: type fixed, parent larm_1, child 25jointt_1, origin xyz=0.0 0.0 0.268085 rpy=0 0 0
- added joint Rigid 35: type fixed, parent transv2_1, child uarm_1, origin xyz=0.0 0.045 0.0651 rpy=0 0 0
- added joint Rigid 37: type fixed, parent uarm_1, child joint14_1, origin xyz=0.0 0.0 0.227 rpy=0 0 0
- added joint Rigid 43: type fixed, parent flange_1, child board_1, origin xyz=0.0 -0.0315 0.0 rpy=0 0 0
- added joint Rigid 44: type fixed, parent board_1, child craw_1, origin xyz=-0.0345 -0.006 0.0595 rpy=0 0 0
- added joint Slider 47: type prismatic, parent craw_1, child crawler_deap12_1, origin xyz=0.063 -0.054 -0.00325 rpy=0 0 0, axis 1.0 -0.0 -0.0, limit lower=-0.01 upper=0.01 effort=100 velocity=100
- added joint Slider 49: type prismatic, parent craw_1, child cralwer_deap_1, origin xyz=0.009 -0.054 -0.00325 rpy=0 0 0, axis 1.0 -0.0 -0.0, limit lower=-0.01 upper=0.01 effort=100 velocity=100
- joint virtual_tip_joint: origin xyz= -0.1 -0.036 -0.00325 rpy=0 0 0 -> xyz= 0.036 -0.054 -0.00325 rpy=0 0 0
